File: Kicad Project/DownconverterPreampModule.sch (KiCad schematic (older format))
At the start: 1 part

Commit message: Initial circuit setup
Parts:
- added C?: C, symbol C
- added R?: R, symbol R
- added RV?: POT, symbol POT
- added U? (x2): LMV751, symbol LMV751
Connections:
- net labels added: GND
- wire segments 0 -> 8
Other:
- moved on the sheet: U?
Changed lines of the file:
@@
 LIBS:contrib
 LIBS:valves
+LIBS:RadarProject
 LIBS:Radar-cache
 EELAYER 25 0
@@
 L MCA1-85L+ U?
 U 1 1 59F14515
-P 7100 4400
-F 0 "U?" H 6550 4760 60  0000 C CNN
-F 1 "MCA1-85L+" H 6760 4870 60  0000 C CNN
-F 2 "" H 7100 4400 60  0001 C CNN
-F 3 "" H 7100 4400 60  0001 C CNN
-	1    7100 4400
+P 3200 5400
+F 0 "U?" H 2650 5760 60  0000 C CNN
+F 1 "MCA1-85L+" H 2860 5870 60  0000 C CNN
+F 2 "" H 3200 5400 60  0001 C CNN
+F 3 "" H 3200 5400 60  0001 C CNN
+	1    3200 5400
+	-1   0    0    -1
+$EndComp
+$Comp
+L LMV751 U?
+U 1 1 59F4A612
+P 5700 4000
+F 0 "U?" H 6050 4550 60  0000 C CNN
+F 1 "LMV751" H 5450 4550 60  0000 C CNN
+F 2 "" H 5700 4000 60  0001 C CNN
+F 3 "" H 5700 4000 60  0001 C CNN
+	1    5700 4000
 	1    0    0    -1
 $EndComp
+$Comp
+L POT RV?
+U 1 1 59F4A697
+P 6650 3000
+F 0 "RV?" V 6475 3000 50  0000 C CNN
+F 1 "POT" V 6550 3000 50  0000 C CNN
+F 2 "" H 6650 3000 50  0001 C CNN
+F 3 "" H 6650 3000 50  0001 C CNN
+	1    6650 3000
+	0    1    1    0
+$EndComp
+$Comp
+L GND #PWR?
+U 1 1 59F4A82A
+P 4950 5050
+F 0 "#PWR?" H 4950 4800 50  0001 C CNN
+F 1 "GND" H 4950 4900 50  0000 C CNN
+F 2 "" H 4950 5050 50  0001 C CNN
+F 3 "" H 4950 5050 50  0001 C CNN
+	1    4950 5050
+	1    0    0    -1
+$EndComp
+$Comp
+L GND #PWR?
+U 1 1 59F4B204
+P 3200 6000
+F 0 "#PWR?" H 3200 5750 50  0001 C CNN
+F 1 "GND" H 3200 5850 50  0000 C CNN
+F 2 "" H 3200 6000 50  0001 C CNN
+F 3 "" H 3200 6000 50  0001 C CNN
+	1    3200 6000
+	1    0    0    -1
+$EndComp
+$Comp
+L R R?
+U 1 1 59F4B291
+P 4550 4300
+F 0 "R?" V 4630 4300 50  0000 C CNN
+F 1 "R" V 4550 4300 50  0000 C CNN
+F 2 "" V 4480 4300 50  0001 C CNN
+F 3 "" H 4550 4300 50  0001 C CNN
+	1    4550 4300
+	0    1    1    0
+$EndComp
+Wire Wire Line
+	3200 4800 3200 4300
+Wire Wire Line
+	3200 4300 4400 4300
+Wire Wire Line
+	4700 4300 5100 4300
+$Comp
+L C C?
+U 1 1 59F4B433
+P 4950 4650
+F 0 "C?" H 4975 4750 50  0000 L CNN
+F 1 "C" H 4975 4550 50  0000 L CNN
+F 2 "" H 4988 4500 50  0001 C CNN
+F 3 "" H 4950 4650 50  0001 C CNN
+	1    4950 4650
+	1    0    0    -1
+$EndComp
+Wire Wire Line
+	4950 4500 4950 4300
+Connection ~ 4950 4300
+Wire Wire Line
+	4950 4800 4950 5050
+Wire Wire Line
+	5100 3000 5100 4000
+Wire Wire Line
+	5100 3000 6500 3000
+Connection ~ 5100 3700
+$Comp
+L LMV751 U?
+U 1 1 59F4B5E2
+P 8400 2700
+F 0 "U?" H 8750 3250 60  0000 C CNN
+F 1 "LMV751" H 8150 3250 60  0000 C CNN
+F 2 "" H 8400 2700 60  0001 C CNN
+F 3 "" H 8400 2700 60  0001 C CNN
+	1    8400 2700
+	1    0    0    -1
+$EndComp
+Wire Wire Line
+	6800 3000 7800 3000
 $EndSCHEMATC

Commit message: Change test
Other:
- note added: "This is a change."
Changed lines of the file:
@@
 Wire Wire Line
 	6800 3000 7800 3000
+Text Notes 4000 2100 0    60   ~ 0
+This is a change.
 $EndSCHEMATC

Commit message: Stuff
Connections:
- wire segments 8 -> 14
Other:
- note added: "INPUT"
- note added: "OUTPUT"
- note removed: "This is a change."
Changed lines of the file:
@@
 Wire Wire Line
 	6800 3000 7800 3000
-Text Notes 4000 2100 0    60   ~ 0
-This is a change.
+Text Notes 2250 5400 0    60   ~ 0
+INPUT
+Text Notes 7350 2400 0    60   ~ 0
+OUTPUT
+Wire Wire Line
+	6300 3700 9850 3700
+Wire Wire Line
+	9850 3700 9850 2400
+Wire Wire Line
+	9850 2400 9000 2400
+$Comp
+L GND #PWR?
+U 1 1 59F7C7AA
+P 7600 4950
+F 0 "#PWR?" H 7600 4700 50  0001 C CNN
+F 1 "GND" H 7600 4800 50  0000 C CNN
+F 2 "" H 7600 4950 50  0001 C CNN
+F 3 "" H 7600 4950 50  0001 C CNN
+	1    7600 4950
+	1    0    0    -1
+$EndComp
+Wire Wire Line
+	7600 2700 7600 4950
+Connection ~ 7600 4300
+Wire Wire Line
+	7600 4300 6300 4300
+Wire Wire Line
+	7600 2700 7800 2700
 $EndSCHEMATC

Commit message: Things.
Connections:
- wire segments 14 -> 18
Other:
- note added: "Gali-1+"
Changed lines of the file:
@@
 	0    1    1    0
 $EndComp
-Wire Wire Line
-	3200 4800 3200 4300
-Wire Wire Line
-	3200 4300 4400 4300
-Wire Wire Line
-	4700 4300 5100 4300
 $Comp
 L C C?
@@
 	1    0    0    -1
 $EndComp
-Wire Wire Line
-	4950 4500 4950 4300
-Connection ~ 4950 4300
-Wire Wire Line
-	4950 4800 4950 5050
-Wire Wire Line
-	5100 3000 5100 4000
-Wire Wire Line
-	5100 3000 6500 3000
-Connection ~ 5100 3700
 $Comp
 L LMV751 U?
@@
 	1    0    0    -1
 $EndComp
-Wire Wire Line
-	6800 3000 7800 3000
 Text Notes 2250 5400 0    60   ~ 0
 INPUT
 Text Notes 7350 2400 0    60   ~ 0
 OUTPUT
-Wire Wire Line
-	6300 3700 9850 3700
-Wire Wire Line
-	9850 3700 9850 2400
-Wire Wire Line
-	9850 2400 9000 2400
 $Comp
 L GND #PWR?
@@
 	1    0    0    -1
 $EndComp
+Text Notes 3900 5400 0    60   ~ 0
+Gali-1+
+Wire Wire Line
+	3200 4800 3200 4300
+Wire Wire Line
+	3200 4300 4400 4300
+Wire Wire Line
+	4700 4300 5100 4300
+Wire Wire Line
+	4950 4500 4950 4300
+Connection ~ 4950 4300
+Wire Wire Line
+	4950 4800 4950 5050
+Wire Wire Line
+	5100 3000 5100 4000
+Wire Wire Line
+	5100 3000 6500 3000
+Connection ~ 5100 3700
+Wire Wire Line
+	6800 3000 7800 3000
+Wire Wire Line
+	6300 3700 9850 3700
+Wire Wire Line
+	9850 3700 9850 2400
+Wire Wire Line
+	9850 2400 9000 2400
 Wire Wire Line
 	7600 2700 7600 4950
@@
 Wire Wire Line
 	7600 2700 7800 2700
+Wire Wire Line
+	7800 2400 7800 1850
+Wire Wire Line
+	7800 1850 9150 1850
+Wire Wire Line
+	9150 1850 9150 3000
+Wire Wire Line
+	9150 3000 9000 3000
 $EndSCHEMATC

Commit message: Added second amplifier.
Parts:
- removed RV?: POT, symbol POT
- added 0.1k, 100k, 10k: R, symbol R
- added C? (x3): 0.1uF, symbol C
- added RV?: POT, symbol POT
- added U?: LMV751, symbol LMV751
- C?: value C -> 270pF
- gave numbers to parts that had none: 1
Connections:
- net labels added: +9V
- wire segments 18 -> 38
Other:
- moved on the sheet: 390k, C?, U?

Commit message: Things.
Parts:
- added C? (x2): C, symbol C
- added U?: GALI-1+, symbol GALI-1+
Connections:
- wire segments 38 -> 41
Other:
- note added: "LO INPUT"
- note added: "RF INPUT"
- note removed: "Gali-1+"
- note removed: "INPUT"
Changed lines of the file:
@@
 	1    0    0    -1
 $EndComp
-Text Notes 1250 6700 0    60   ~ 0
-INPUT
+Text Notes 1100 6700 0    60   ~ 0
+RF INPUT
 Text Notes 3150 2450 0    60   ~ 0
 OUTPUT
-Text Notes 2900 6700 0    60   ~ 0
-Gali-1+
 Wire Wire Line
 	2200 6100 2200 5600
@@
 Connection ~ 8000 4300
 Connection ~ 6800 3700
+$Comp
+L GALI-1+ U?
+U 1 1 59F927C1
+P 5100 6700
+F 0 "U?" H 5500 7250 60  0000 C CNN
+F 1 "GALI-1+" H 4800 7250 60  0000 C CNN
+F 2 "" H 5100 6700 60  0001 C CNN
+F 3 "" H 5100 6700 60  0001 C CNN
+	1    5100 6700
+	-1   0    0    -1
+$EndComp
+$Comp
+L GND #PWR?
+U 1 1 59F92916
+P 5100 7150
+F 0 "#PWR?" H 5100 6900 50  0001 C CNN
+F 1 "GND" H 5100 7000 50  0000 C CNN
+F 2 "" H 5100 7150 50  0001 C CNN
+F 3 "" H 5100 7150 50  0001 C CNN
+	1    5100 7150
+	1    0    0    -1
+$EndComp
+Text Notes 6300 6750 0    60   ~ 0
+LO INPUT
+$Comp
+L C C?
+U 1 1 59F92971
+P 4150 6700
+F 0 "C?" H 4175 6800 50  0000 L CNN
+F 1 "C" H 4175 6600 50  0000 L CNN
+F 2 "" H 4188 6550 50  0001 C CNN
+F 3 "" H 4150 6700 50  0001 C CNN
+	1    4150 6700
+	0    1    1    0
+$EndComp
+$Comp
+L C C?
+U 1 1 59F92A41
+P 6050 6700
+F 0 "C?" H 6075 6800 50  0000 L CNN
+F 1 "C" H 6075 6600 50  0000 L CNN
+F 2 "" H 6088 6550 50  0001 C CNN
+F 3 "" H 6050 6700 50  0001 C CNN
+	1    6050 6700
+	0    1    1    0
+$EndComp
+Wire Wire Line
+	5900 6700 5800 6700
+Wire Wire Line
+	4300 6700 4400 6700
+Wire Wire Line
+	4000 6700 2800 6700
 $EndSCHEMATC

Commit message: Reorganization
Parts:
- removed 0.1k, 100k, 10k, 390k: R, symbol R
- removed C?: 270pF, symbol C
- removed C? (x3): 0.1uF, symbol C
- removed C? (x2): C, symbol C
- removed RV?: POT, symbol POT
- removed U?: MCA1-85L+, symbol MCA1-85L+
- removed U? (x3): LMV751, symbol LMV751
- removed U?: GALI-1+, symbol GALI-1+
- added C1, C2, C3, C4: 270pF, symbol C
- added R1, R2: 75, symbol R
- added R3: 390k, symbol R
- added R4: 100, symbol R
- added R5: 100k, symbol R
- added R6: 10k, symbol R
- added RV1: POT, symbol POT
- added U1: GALI-1+, symbol GALI-1+
- added U2: MCA1-85L+, symbol MCA1-85L+
- added U3, U4, U5: LMV751, symbol LMV751
Connections:
- wire segments 41 -> 44
Other:
- note added: "LO Input"
- note added: "Low-Pass Filter"
- note added: "RF Input"
- note removed: "LO INPUT"
- note removed: "RF INPUT"

Commit message: PCB 1
Parts:
- C1, C2, C3, C4: footprint (none) -> Capacitors_SMD:C_0603
- R1, R2, R3, R4, R5, R6: footprint (none) -> Resistors_SMD:R_0603
Connections:
- wire segments 44 -> 45
Other:
- moved on the sheet: R1, R2
Changed lines of the file:
@@
 F 0 "C1" H 1425 3900 50  0000 L CNN
 F 1 "270pF" H 1425 3700 50  0000 L CNN
-F 2 "" H 1438 3650 50  0001 C CNN
+F 2 "Capacitors_SMD:C_0603" H 1438 3650 50  0001 C CNN
 F 3 "" H 1400 3800 50  0001 C CNN
 	1    1400 3800
@@
 $EndComp
 $Comp
-L GND #PWR09
+L GND #PWR015
 U 1 1 59FB8769
 P 2250 4250
-F 0 "#PWR09" H 2250 4000 50  0001 C CNN
+F 0 "#PWR015" H 2250 4000 50  0001 C CNN
 F 1 "GND" H 2250 4100 50  0000 C CNN
 F 2 "" H 2250 4250 50  0001 C CNN
@@
 F 0 "C3" H 3625 3900 50  0000 L CNN
 F 1 "270pF" H 3625 3700 50  0000 L CNN
-F 2 "" H 3638 3650 50  0001 C CNN
+F 2 "Capacitors_SMD:C_0603" H 3638 3650 50  0001 C CNN
 F 3 "" H 3600 3800 50  0001 C CNN
 	1    3600 3800
@@
 F 0 "C2" H 3225 3400 50  0000 L CNN
 F 1 "270pF" H 3225 3200 50  0000 L CNN
-F 2 "" H 3238 3150 50  0001 C CNN
+F 2 "Capacitors_SMD:C_0603" H 3238 3150 50  0001 C CNN
 F 3 "" H 3200 3300 50  0001 C CNN
 	1    3200 3300
@@
 L R R1
 U 1 1 59FB88C3
-P 3100 2800
-F 0 "R1" V 3180 2800 50  0000 C CNN
-F 1 "75" V 3100 2800 50  0000 C CNN
-F 2 "" V 3030 2800 50  0001 C CNN
-F 3 "" H 3100 2800 50  0001 C CNN
-	1    3100 2800
-	0    1    1    0
+P 2900 3550
+F 0 "R1" V 2980 3550 50  0000 C CNN
+F 1 "75" V 2900 3550 50  0000 C CNN
+F 2 "Resistors_SMD:R_0603" V 2830 3550 50  0001 C CNN
+F 3 "" H 2900 3550 50  0001 C CNN
+	1    2900 3550
+	1    0    0    -1
 $EndComp
 $Comp
 L R R2
 U 1 1 59FB89F7
-P 3400 2800
-F 0 "R2" V 3480 2800 50  0000 C CNN
-F 1 "75" V 3400 2800 50  0000 C CNN
-F 2 "" V 3330 2800 50  0001 C CNN
-F 3 "" H 3400 2800 50  0001 C CNN
-	1    3400 2800
-	0    1    1    0
-$EndComp
-Wire Wire Line
-	2900 3800 2900 2800
-Wire Wire Line
-	2900 2800 2950 2800
+P 3250 2800
+F 0 "R2" V 3330 2800 50  0000 C CNN
+F 1 "75" V 3250 2800 50  0000 C CNN
+F 2 "Resistors_SMD:R_0603" V 3180 2800 50  0001 C CNN
+F 3 "" H 3250 2800 50  0001 C CNN
+	1    3250 2800
+	0    1    1    0
+$EndComp
 Connection ~ 2900 3800
 Connection ~ 2900 3300
 $Comp
-L +9V #PWR010
+L +9V #PWR016
 U 1 1 59FB8AD6
-P 3650 2600
-F 0 "#PWR010" H 3650 2450 50  0001 C CNN
-F 1 "+9V" H 3650 2740 50  0000 C CNN
-F 2 "" H 3650 2600 50  0001 C CNN
-F 3 "" H 3650 2600 50  0001 C CNN
-	1    3650 2600
-	1    0    0    -1
-$EndComp
-$Comp
-L GND #PWR011
+P 3600 2600
+F 0 "#PWR016" H 3600 2450 50  0001 C CNN
+F 1 "+9V" H 3600 2740 50  0000 C CNN
+F 2 "" H 3600 2600 50  0001 C CNN
+F 3 "" H 3600 2600 50  0001 C CNN
+	1    3600 2600
+	1    0    0    -1
+$EndComp
+$Comp
+L GND #PWR017
 U 1 1 59FB8AF6
 P 3450 3400
-F 0 "#PWR011" H 3450 3150 50  0001 C CNN
+F 0 "#PWR017" H 3450 3150 50  0001 C CNN
 F 1 "GND" H 3450 3250 50  0000 C CNN
 F 2 "" H 3450 3400 50  0001 C CNN
@@
 $EndComp
 Wire Wire Line
-	3550 2800 3650 2800
-Wire Wire Line
-	3650 2800 3650 2600
+	3600 2800 3600 2600
 Wire Wire Line
 	3350 3300 3450 3300
@@
 	5450 5100 5450 3800
 $Comp
-L GND #PWR012
+L GND #PWR018
 U 1 1 59FB8C63
 P 4850 4400
-F 0 "#PWR012" H 4850 4150 50  0001 C CNN
+F 0 "#PWR018" H 4850 4150 50  0001 C CNN
 F 1 "GND" H 4850 4250 50  0000 C CNN
 F 2 "" H 4850 4400 50  0001 C CNN
@@
 F 0 "R3" V 5280 2800 50  0000 C CNN
 F 1 "390k" V 5200 2800 50  0000 C CNN
-F 2 "" V 5130 2800 50  0001 C CNN
+F 2 "Resistors_SMD:R_0603" V 5130 2800 50  0001 C CNN
 F 3 "" H 5200 2800 50  0001 C CNN
 	1    5200 2800
@@
 F 0 "C4" H 5575 3150 50  0000 L CNN
 F 1 "270pF" H 5575 2950 50  0000 L CNN
-F 2 "" H 5588 2900 50  0001 C CNN
+F 2 "Capacitors_SMD:C_0603" H 5588 2900 50  0001 C CNN
 F 3 "" H 5550 3050 50  0001 C CNN
 	1    5550 3050
@@
 	5550 3200 5550 3300
 $Comp
-L GND #PWR013
+L GND #PWR019
 U 1 1 59FB902C
 P 5550 3300
-F 0 "#PWR013" H 5550 3050 50  0001 C CNN
+F 0 "#PWR019" H 5550 3050 50  0001 C CNN
 F 1 "GND" H 5550 3150 50  0000 C CNN
 F 2 "" H 5550 3300 50  0001 C CNN
@@
 	5650 2200 5750 2200
 $Comp
-L +9V #PWR014
+L +9V #PWR020
 U 1 1 59FB90DA
 P 7000 2150
-F 0 "#PWR014" H 7000 2000 50  0001 C CNN
+F 0 "#PWR020" H 7000 2000 50  0001 C CNN
 F 1 "+9V" H 7000 2290 50  0000 C CNN
 F 2 "" H 7000 2150 50  0001 C CNN
@@
 $EndComp
 $Comp
-L GND #PWR015
+L GND #PWR021
 U 1 1 59FB910C
 P 7000 2850
-F 0 "#PWR015" H 7000 2600 50  0001 C CNN
+F 0 "#PWR021" H 7000 2600 50  0001 C CNN
 F 1 "GND" H 7000 2700 50  0000 C CNN
 F 2 "" H 7000 2850 50  0001 C CNN
@@
 F 0 "R4" V 7380 2800 50  0000 C CNN
 F 1 "100" V 7300 2800 50  0000 C CNN
-F 2 "" V 7230 2800 50  0001 C CNN
+F 2 "Resistors_SMD:R_0603" V 7230 2800 50  0001 C CNN
 F 3 "" H 7300 2800 50  0001 C CNN
 	1    7300 2800
@@
 Connection ~ 5650 2200
 $Comp
-L GND #PWR016
+L GND #PWR022
 U 1 1 59FB957B
 P 7650 2500
-F 0 "#PWR016" H 7650 2250 50  0001 C CNN
+F 0 "#PWR022" H 7650 2250 50  0001 C CNN
 F 1 "GND" H 7650 2350 50  0000 C CNN
 F 2 "" H 7650 2500 50  0001 C CNN
@@
 $EndComp
 $Comp
-L GND #PWR017
+L GND #PWR023
 U 1 1 59FB95A7
 P 8950 2900
-F 0 "#PWR017" H 8950 2650 50  0001 C CNN
+F 0 "#PWR023" H 8950 2650 50  0001 C CNN
 F 1 "GND" H 8950 2750 50  0000 C CNN
 F 2 "" H 8950 2900 50  0001 C CNN
@@
 $EndComp
 $Comp
-L +9V #PWR018
+L +9V #PWR024
 U 1 1 59FB95D3
 P 8950 2100
-F 0 "#PWR018" H 8950 1950 50  0001 C CNN
+F 0 "#PWR024" H 8950 1950 50  0001 C CNN
 F 1 "+9V" H 8950 2240 50  0000 C CNN
 F 2 "" H 8950 2100 50  0001 C CNN
@@
 F 0 "R5" V 7580 2450 50  0000 C CNN
 F 1 "100k" V 7500 2450 50  0000 C CNN
-F 2 "" V 7430 2450 50  0001 C CNN
+F 2 "Resistors_SMD:R_0603" V 7430 2450 50  0001 C CNN
 F 3 "" H 7500 2450 50  0001 C CNN
 	1    7500 2450
@@
 $EndComp
 $Comp
-L +9V #PWR019
+L +9V #PWR025
 U 1 1 59FB9877
 P 10850 2100
-F 0 "#PWR019" H 10850 1950 50  0001 C CNN
+F 0 "#PWR025" H 10850 1950 50  0001 C CNN
 F 1 "+9V" H 10850 2240 50  0000 C CNN
 F 2 "" H 10850 2100 50  0001 C CNN
@@
 $EndComp
 $Comp
-L GND #PWR020
+L GND #PWR026
 U 1 1 59FB98A7
 P 10850 2900
-F 0 "#PWR020" H 10850 2650 50  0001 C CNN
+F 0 "#PWR026" H 10850 2650 50  0001 C CNN
 F 1 "GND" H 10850 2750 50  0000 C CNN
 F 2 "" H 10850 2900 50  0001 C CNN
@@
 $EndComp
 $Comp
-L GND #PWR021
+L GND #PWR027
 U 1 1 59FB98E5
 P 9550 2500
-F 0 "#PWR021" H 9550 2250 50  0001 C CNN
+F 0 "#PWR027" H 9550 2250 50  0001 C CNN
 F 1 "GND" H 9550 2350 50  0000 C CNN
 F 2 "" H 9550 2500 50  0001 C CNN
@@
 F 0 "R6" V 9480 2450 50  0000 C CNN
 F 1 "10k" V 9400 2450 50  0000 C CNN
-F 2 "" V 9330 2450 50  0001 C CNN
+F 2 "Resistors_SMD:R_0603" V 9330 2450 50  0001 C CNN
 F 3 "" H 9400 2450 50  0001 C CNN
 	1    9400 2450
@@
 Text Notes 10800 1400 0    60   ~ 0
 OUTPUT
+Wire Wire Line
+	2900 3800 2900 3700
+Wire Wire Line
+	2900 2800 2900 3400
+Wire Wire Line
+	2900 2800 3100 2800
+Wire Wire Line
+	3400 2800 3600 2800
 $EndSCHEMATC
