File: Kicad Project/DownconverterPreampModule.sch (KiCad schematic (older format))
At the start: 13 parts, among them U1 GALI-1+, U2 MCA1-85L+, U4 LMV751, U5 LMV751

Commit message: PCB LAYOUT update
Parts:
- R1, R2: footprint Resistors_SMD:R_0603 -> RadarComponents:100PAD
Connections:
- net at C3.2, U1.3 (RF_OUT): now also R1.2
- net LO renamed PowerSplitter
Changed lines of the file:
@@
 $EndComp
 $Comp
-L GND #PWR019
+L GND #PWR01
 U 1 1 59FB8769
 P 2250 4250
-F 0 "#PWR019" H 2250 4000 50  0001 C CNN
+F 0 "#PWR01" H 2250 4000 50  0001 C CNN
 F 1 "GND" H 2250 4100 50  0000 C CNN
 F 2 "" H 2250 4250 50  0001 C CNN
@@
 F 0 "R1" V 2980 3550 50  0000 C CNN
 F 1 "75" V 2900 3550 50  0000 C CNN
-F 2 "Resistors_SMD:R_0603" V 2830 3550 50  0001 C CNN
+F 2 "RadarComponents:100PAD" V 2830 3550 50  0001 C CNN
 F 3 "" H 2900 3550 50  0001 C CNN
 	1    2900 3550
@@
 F 0 "R2" V 3330 2800 50  0000 C CNN
 F 1 "75" V 3250 2800 50  0000 C CNN
-F 2 "Resistors_SMD:R_0603" V 3180 2800 50  0001 C CNN
+F 2 "RadarComponents:100PAD" V 3180 2800 50  0001 C CNN
 F 3 "" H 3250 2800 50  0001 C CNN
 	1    3250 2800
 	0    1    1    0
 $EndComp
-Connection ~ 2900 3800
+Connection ~ 3050 3800
 Connection ~ 2900 3300
 $Comp
-L +9V #PWR020
+L +9V #PWR02
 U 1 1 59FB8AD6
 P 3600 2600
-F 0 "#PWR020" H 3600 2450 50  0001 C CNN
+F 0 "#PWR02" H 3600 2450 50  0001 C CNN
 F 1 "+9V" H 3600 2740 50  0000 C CNN
 F 2 "" H 3600 2600 50  0001 C CNN
@@
 $EndComp
 $Comp
-L GND #PWR021
+L GND #PWR03
 U 1 1 59FB8AF6
 P 3450 3400
-F 0 "#PWR021" H 3450 3150 50  0001 C CNN
+F 0 "#PWR03" H 3450 3150 50  0001 C CNN
 F 1 "GND" H 3450 3250 50  0000 C CNN
 F 2 "" H 3450 3400 50  0001 C CNN
@@
 	5450 5100 5450 3800
 $Comp
-L GND #PWR022
+L GND #PWR04
 U 1 1 59FB8C63
 P 4850 4400
-F 0 "#PWR022" H 4850 4150 50  0001 C CNN
+F 0 "#PWR04" H 4850 4150 50  0001 C CNN
 F 1 "GND" H 4850 4250 50  0000 C CNN
 F 2 "" H 4850 4400 50  0001 C CNN
@@
 $EndComp
 $Comp
-L GND #PWR023
+L GND #PWR05
 U 1 1 59FB957B
 P 7650 2500
-F 0 "#PWR023" H 7650 2250 50  0001 C CNN
+F 0 "#PWR05" H 7650 2250 50  0001 C CNN
 F 1 "GND" H 7650 2350 50  0000 C CNN
 F 2 "" H 7650 2500 50  0001 C CNN
@@
 $EndComp
 $Comp
-L GND #PWR024
+L GND #PWR06
 U 1 1 59FB95A7
 P 8950 2900
-F 0 "#PWR024" H 8950 2650 50  0001 C CNN
+F 0 "#PWR06" H 8950 2650 50  0001 C CNN
 F 1 "GND" H 8950 2750 50  0000 C CNN
 F 2 "" H 8950 2900 50  0001 C CNN
@@
 $EndComp
 $Comp
-L +9V #PWR025
+L +9V #PWR07
 U 1 1 59FB95D3
 P 8950 2100
-F 0 "#PWR025" H 8950 1950 50  0001 C CNN
+F 0 "#PWR07" H 8950 1950 50  0001 C CNN
 F 1 "+9V" H 8950 2240 50  0000 C CNN
 F 2 "" H 8950 2100 50  0001 C CNN
@@
 $EndComp
 $Comp
-L +9V #PWR026
+L +9V #PWR08
 U 1 1 59FB9877
 P 10850 2100
-F 0 "#PWR026" H 10850 1950 50  0001 C CNN
+F 0 "#PWR08" H 10850 1950 50  0001 C CNN
 F 1 "+9V" H 10850 2240 50  0000 C CNN
 F 2 "" H 10850 2100 50  0001 C CNN
@@
 $EndComp
 $Comp
-L GND #PWR027
+L GND #PWR09
 U 1 1 59FB98A7
 P 10850 2900
-F 0 "#PWR027" H 10850 2650 50  0001 C CNN
+F 0 "#PWR09" H 10850 2650 50  0001 C CNN
 F 1 "GND" H 10850 2750 50  0000 C CNN
 F 2 "" H 10850 2900 50  0001 C CNN
@@
 $EndComp
 $Comp
-L GND #PWR028
+L GND #PWR010
 U 1 1 59FB98E5
 P 9550 2500
-F 0 "#PWR028" H 9550 2250 50  0001 C CNN
+F 0 "#PWR010" H 9550 2250 50  0001 C CNN
 F 1 "GND" H 9550 2350 50  0000 C CNN
 F 2 "" H 9550 2500 50  0001 C CNN
@@
 OUTPUT
 Wire Wire Line
-	2900 3800 2900 3700
-Wire Wire Line
 	2900 2800 2900 3400
 Wire Wire Line
@@
 Text Notes 5200 3050 0    60   Italic 0
 0.23737 inch single pole filter
-Text HLabel 800  3800 0    60   Input ~ 0
-LO
-Text HLabel 1250 5100 0    60   Input ~ 0
+Wire Wire Line
+	1250 3800 800  3800
+Text GLabel 800  3800 0    60   Input ~ 0
+PowerSplitter
+Text GLabel 1250 5100 0    60   Input ~ 0
 RFIN
-Text Label 800  3800 0    60   ~ 0
-PowerSplitter
-Wire Wire Line
-	1250 3800 800  3800
+Wire Wire Line
+	2900 3700 3050 3700
+Wire Wire Line
+	3050 3700 3050 3800
 $EndSCHEMATC

Commit message: PCB
Parts:
- removed RV1: POT, symbol POT
- removed U5: LMV751, RadarComponents:SOT23-5, symbol LMV751
- added C15, C16, C4: 270pF, Capacitors_SMD:C_0603, symbol C
- added R3: 47k, Resistors_SMD:R_0603, symbol R
- R4: value 100 -> 10k
- R5: value 100k -> 100
- R6: value 10k -> 100k
Connections:
- net +9V: now also C16.1, R3.1
- net GND: now also R4.2, C16.2, C4.2; no longer U4.4 (VIN-)
- net at U2.3 (IF): now also C15.2; no longer R4.2
- net at U4.1 (VOUT): now also R6.2; no longer R5.1
- net at R4.1, U4.3 (VIN+): now also C4.1, R3.2; no longer R5.2
- net at R6.1: now also R5.1, U4.4 (VIN-)
- new net: C15.1, R5.2
Other:
- note added: "OUT"
- note removed: "OUTPUT"
- moved on the sheet: U4
