File: Kicad Project/SourceModule.sch (KiCad schematic (older format))
At the start: 22 parts, among them U6 GALI-2+, U7 RMK-3-93+, U8 GALI-2+

Commit message: PCB LAYOUT update
Parts:
- added J1, J2, J3, J4: Conn_01x02, symbol Conn_01x02
Connections:
- net labels added: Filter
- net labels removed: LO, TX
- wire segments 44 -> 47
Other:
- moved on the sheet: .1uF3, .1uF4, C9, R13, R14, U8

Commit message: Added Filters to PCB
Parts:
- MS1: footprint (none) -> RadarComponents:powersplitter2
Connections:
- net PowerSplitter: now also MS1.2 (OUT1), MS1.3 (OUT2); no longer .1uF4.1
- net at MS1.1 (Input): now also .1uF4.1
Changed lines of the file:
@@
 F 0 "MS1" H 8260 6100 60  0000 C CNN
 F 1 "PowerDivider" H 7640 6100 60  0000 C CNN
-F 2 "" H 7850 5550 60  0001 C CNN
+F 2 "RadarComponents:powersplitter2" H 7850 5550 60  0001 C CNN
 F 3 "" H 7850 5550 60  0001 C CNN
 	1    7850 5550
@@
 	8200 2200 8200 2050
 Connection ~ 8200 2200
-Text GLabel 10700 3850 2    60   Input ~ 0
-PowerSplitter
 $Comp
 L Conn_01x02 J4
@@
 Wire Wire Line
 	2050 4750 2400 4750
+Wire Wire Line
+	6800 5550 7150 5550
+Text GLabel 8550 5300 2    60   Input ~ 0
+PowerSplitter
+Text GLabel 8550 5800 2    60   Input ~ 0
+PowerSplitter
 $EndSCHEMATC

Commit message: PCB Changes
Parts:
- added C17: 10uF, Capacitors_SMD:C_0805, symbol C
- added C19: C, Capacitors_SMD:C_0805, symbol C
- added J5: Conn_01x02, Pin_Headers:Pin_Header_Straight_1x02_Pitch1.27mm, symbol Conn_01x02
- added R15, R20: R, Resistors_SMD:R_0603, symbol R
- added U5: AP1117-50, RadarComponents:ZLDO1117, symbol AP1117-50
- C8, C9: footprint RadarComponents:100PAD -> RadarComponents:100PAD+GND2
- J1, J2, J3: footprint (none) -> Pin_Headers:Pin_Header_Straight_1x02_Pitch1.27mm
- J4: footprint (none) -> RadarComponents:UFL
- renumbered .1uF1 to C18, .1uF2 to C20, .1uF3 to C21
Connections:
- net +9V: now also C17.1, U5.3 (VI)
- net GND: now also C17.2, C19.2, J5.1 (Pin_1), R15.2
- new net: R15.1, R20.2, U5.1 (GND)
- new net +5V: C19.1, J5.2 (Pin_2), R20.1, U5.2 (VO)
Other:
- note added: "3.3V from Teensy"
- note added: "5V from Regulator to Teensy"
- note added: "9V from Battery\n"
- moved on the sheet: J4

Commit message: More PCB Updates
Parts:
- R14, R8: footprint RadarComponents:100PAD -> RadarComponents:100PAD+GND
Changed lines of the file:
@@
 F 0 "R8" V 5480 1300 50  0000 C CNN
 F 1 "75" V 5400 1300 50  0000 C CNN
-F 2 "RadarComponents:100PAD" V 5330 1300 50  0001 C CNN
+F 2 "RadarComponents:100PAD+GND" V 5330 1300 50  0001 C CNN
 F 3 "" H 5400 1300 50  0001 C CNN
 	1    5400 1300
@@
 F 0 "R14" V 10380 1300 50  0000 C CNN
 F 1 "75" V 10300 1300 50  0000 C CNN
-F 2 "RadarComponents:100PAD" V 10230 1300 50  0001 C CNN
+F 2 "RadarComponents:100PAD+GND" V 10230 1300 50  0001 C CNN
 F 3 "" H 10300 1300 50  0001 C CNN
 	1    10300 1300

Commit message: PCB Pre Flood
Parts:
- added J7: Conn_01x02, Pin_Headers:Pin_Header_Straight_1x02_Pitch1.27mm, symbol Conn_01x02
Connections:
- net GND: now also J7.1 (Pin_1)
- net at VCO1.4 (~SHDN): now also J7.2 (Pin_2)
Changed lines of the file:
@@
 Text Notes 2750 5400 0    60   ~ 0
 5V from Regulator to Teensy
+$Comp
+L Conn_01x02 J7
+U 1 1 5A051D07
+P 1300 2900
+F 0 "J7" H 1300 3000 50  0000 C CNN
+F 1 "Conn_01x02" H 1300 2700 50  0000 C CNN
+F 2 "Pin_Headers:Pin_Header_Straight_1x02_Pitch1.27mm" H 1300 2900 50  0001 C CNN
+F 3 "" H 1300 2900 50  0001 C CNN
+	1    1300 2900
+	-1   0    0    1
+$EndComp
+$Comp
+L GND #PWR047
+U 1 1 5A051D90
+P 1500 2900
+F 0 "#PWR047" H 1500 2650 50  0001 C CNN
+F 1 "GND" H 1500 2750 50  0000 C CNN
+F 2 "" H 1500 2900 50  0001 C CNN
+F 3 "" H 1500 2900 50  0001 C CNN
+	1    1500 2900
+	1    0    0    -1
+$EndComp
 $EndSCHEMATC
