File: Kicad Project/SourceModule.sch (KiCad schematic (older format))
At the start: 29 parts, among them J2 CONN_02X06, U16 TC1185, U17 MAX2752, U18 ufl, U19 ufl, U5 AP1117-50, U6 LEE-39+, U7 RMK-3-93+, U8 GALI-2+

Commit message: Damian's almost to rev 2 completion, needs audio amps
Parts:
- C8, C9: footprint RadarComponents:100PAD+GND2 -> RadarComponents:100PAD+GND3
Changed lines of the file:
@@
 $EndComp
 $Comp
-L +3.3V #PWR020
+L +3.3V #PWR027
 U 1 1 59F4A689
 P 3400 2550
-F 0 "#PWR020" H 3400 2400 50  0001 C CNN
+F 0 "#PWR027" H 3400 2400 50  0001 C CNN
 F 1 "+3.3V" H 3400 2690 50  0000 C CNN
 F 2 "" H 3400 2550 50  0001 C CNN
@@
 $EndComp
 $Comp
-L GND #PWR021
+L GND #PWR028
 U 1 1 59F4A990
 P 1050 1800
-F 0 "#PWR021" H 1050 1550 50  0001 C CNN
+F 0 "#PWR028" H 1050 1550 50  0001 C CNN
 F 1 "GND" H 1050 1650 50  0000 C CNN
 F 2 "" H 1050 1800 50  0001 C CNN
@@
 $EndComp
 $Comp
-L GND #PWR022
+L GND #PWR029
 U 1 1 59F4AA4C
 P 3200 3250
-F 0 "#PWR022" H 3200 3000 50  0001 C CNN
+F 0 "#PWR029" H 3200 3000 50  0001 C CNN
 F 1 "GND" H 3200 3100 50  0000 C CNN
 F 2 "" H 3200 3250 50  0001 C CNN
@@
 $EndComp
 $Comp
-L GND #PWR023
+L GND #PWR030
 U 1 1 59F4AA6C
 P 3600 3250
-F 0 "#PWR023" H 3600 3000 50  0001 C CNN
+F 0 "#PWR030" H 3600 3000 50  0001 C CNN
 F 1 "GND" H 3600 3100 50  0000 C CNN
 F 2 "" H 3600 3250 50  0001 C CNN
@@
 	3600 2600 3600 2950
 $Comp
-L GND #PWR024
+L GND #PWR031
 U 1 1 59F4AB52
 P 3150 1700
-F 0 "#PWR024" H 3150 1450 50  0001 C CNN
+F 0 "#PWR031" H 3150 1450 50  0001 C CNN
 F 1 "GND" H 3150 1550 50  0000 C CNN
 F 2 "" H 3150 1700 50  0001 C CNN
@@
 $EndComp
 $Comp
-L GND #PWR025
+L GND #PWR032
 U 1 1 59F4AE46
 P 850 2650
-F 0 "#PWR025" H 850 2400 50  0001 C CNN
+F 0 "#PWR032" H 850 2400 50  0001 C CNN
 F 1 "GND" H 850 2500 50  0000 C CNN
 F 2 "" H 850 2650 50  0001 C CNN
@@
 Frequency Feedback
 $Comp
-L GND #PWR026
+L GND #PWR033
 U 1 1 59F4B365
 P 7300 2900
-F 0 "#PWR026" H 7300 2650 50  0001 C CNN
+F 0 "#PWR033" H 7300 2650 50  0001 C CNN
 F 1 "GND" H 7300 2750 50  0000 C CNN
 F 2 "" H 7300 2900 50  0001 C CNN
@@
 $EndComp
 $Comp
-L GND #PWR027
+L GND #PWR034
 U 1 1 59F9EB1B
 P 4750 2650
-F 0 "#PWR027" H 4750 2400 50  0001 C CNN
+F 0 "#PWR034" H 4750 2400 50  0001 C CNN
 F 1 "GND" H 4750 2500 50  0000 C CNN
 F 2 "" H 4750 2650 50  0001 C CNN
@@
 	6150 1300 6150 1150
 $Comp
-L +9V #PWR028
+L +9V #PWR035
 U 1 1 59F9EF36
 P 6150 1150
-F 0 "#PWR028" H 6150 1000 50  0001 C CNN
+F 0 "#PWR035" H 6150 1000 50  0001 C CNN
 F 1 "+9V" H 6150 1290 50  0000 C CNN
 F 2 "" H 6150 1150 50  0001 C CNN
@@
 $EndComp
 $Comp
-L GND #PWR029
+L GND #PWR036
 U 1 1 59F9EFD4
 P 5950 1750
-F 0 "#PWR029" H 5950 1500 50  0001 C CNN
+F 0 "#PWR036" H 5950 1500 50  0001 C CNN
 F 1 "GND" H 5950 1600 50  0000 C CNN
 F 2 "" H 5950 1750 50  0001 C CNN
@@
 F 0 "C8" H 5675 1800 50  0000 L CNN
 F 1 "C" H 5675 1600 50  0000 L CNN
-F 2 "RadarComponents:100PAD+GND2" H 5688 1550 50  0001 C CNN
+F 2 "RadarComponents:100PAD+GND3" H 5688 1550 50  0001 C CNN
 F 3 "" H 5650 1700 50  0001 C CNN
 	1    5650 1700
@@
 	10700 1300 10700 1150
 $Comp
-L +9V #PWR030
+L +9V #PWR037
 U 1 1 59F9F432
 P 10700 1150
-F 0 "#PWR030" H 10700 1000 50  0001 C CNN
+F 0 "#PWR037" H 10700 1000 50  0001 C CNN
 F 1 "+9V" H 10700 1290 50  0000 C CNN
 F 2 "" H 10700 1150 50  0001 C CNN
@@
 $EndComp
 $Comp
-L GND #PWR031
+L GND #PWR038
 U 1 1 59F9F438
 P 10500 1750
-F 0 "#PWR031" H 10500 1500 50  0001 C CNN
+F 0 "#PWR038" H 10500 1500 50  0001 C CNN
 F 1 "GND" H 10500 1600 50  0000 C CNN
 F 2 "" H 10500 1750 50  0001 C CNN
@@
 F 0 "C9" H 10275 1800 50  0000 L CNN
 F 1 "C" H 10275 1600 50  0000 L CNN
-F 2 "RadarComponents:100PAD+GND2" H 10288 1550 50  0001 C CNN
+F 2 "RadarComponents:100PAD+GND3" H 10288 1550 50  0001 C CNN
 F 3 "" H 10250 1700 50  0001 C CNN
 	1    10250 1700
@@
 $EndComp
 $Comp
-L GND #PWR032
+L GND #PWR039
 U 1 1 59F9F88B
 P 9350 2650
-F 0 "#PWR032" H 9350 2400 50  0001 C CNN
+F 0 "#PWR039" H 9350 2400 50  0001 C CNN
 F 1 "GND" H 9350 2500 50  0000 C CNN
 F 2 "" H 9350 2650 50  0001 C CNN
@@
 	8000 2200 8350 2200
 $Comp
-L GND #PWR033
+L GND #PWR040
 U 1 1 5A020DEA
 P 8200 2200
-F 0 "#PWR033" H 8200 1950 50  0001 C CNN
+F 0 "#PWR040" H 8200 1950 50  0001 C CNN
 F 1 "GND" H 8200 2050 50  0000 C CNN
 F 2 "" H 8200 2200 50  0001 C CNN
@@
 Connection ~ 8200 2200
 $Comp
-L +3.3V #PWR034
+L +3.3V #PWR041
 U 1 1 5A027182
 P 2350 4350
-F 0 "#PWR034" H 2350 4200 50  0001 C CNN
+F 0 "#PWR041" H 2350 4200 50  0001 C CNN
 F 1 "+3.3V" H 2350 4490 50  0000 C CNN
 F 2 "" H 2350 4350 50  0001 C CNN
@@
 $EndComp
 $Comp
-L +9V #PWR035
+L +9V #PWR042
 U 1 1 5A027267
 P 2650 4550
-F 0 "#PWR035" H 2650 4400 50  0001 C CNN
+F 0 "#PWR042" H 2650 4400 50  0001 C CNN
 F 1 "+9V" H 2650 4690 50  0000 C CNN
 F 2 "" H 2650 4550 50  0001 C CNN
@@
 $EndComp
 $Comp
-L +5V #PWR036
+L +5V #PWR043
 U 1 1 5A04CEA6
 P 3800 5900
-F 0 "#PWR036" H 3800 5750 50  0001 C CNN
+F 0 "#PWR043" H 3800 5750 50  0001 C CNN
 F 1 "+5V" H 3800 6040 50  0000 C CNN
 F 2 "" H 3800 5900 50  0001 C CNN
@@
 Connection ~ 2000 5900
 $Comp
-L GND #PWR037
+L GND #PWR044
 U 1 1 5A04D587
 P 3550 6250
-F 0 "#PWR037" H 3550 6000 50  0001 C CNN
+F 0 "#PWR044" H 3550 6000 50  0001 C CNN
 F 1 "GND" H 3550 6100 50  0000 C CNN
 F 2 "" H 3550 6250 50  0001 C CNN
@@
 $EndComp
 $Comp
-L GND #PWR038
+L GND #PWR045
 U 1 1 5A04D65D
 P 2650 6350
-F 0 "#PWR038" H 2650 6100 50  0001 C CNN
+F 0 "#PWR045" H 2650 6100 50  0001 C CNN
 F 1 "GND" H 2650 6200 50  0000 C CNN
 F 2 "" H 2650 6350 50  0001 C CNN
@@
 $EndComp
 $Comp
-L GND #PWR039
+L GND #PWR046
 U 1 1 5A04D6C5
 P 2000 6300
-F 0 "#PWR039" H 2000 6050 50  0001 C CNN
+F 0 "#PWR046" H 2000 6050 50  0001 C CNN
 F 1 "GND" H 2000 6150 50  0000 C CNN
 F 2 "" H 2000 6300 50  0001 C CNN
@@
 $EndComp
 $Comp
-L +9V #PWR040
+L +9V #PWR047
 U 1 1 5A04DB89
 P 1750 5900
-F 0 "#PWR040" H 1750 5750 50  0001 C CNN
+F 0 "#PWR047" H 1750 5750 50  0001 C CNN
 F 1 "+9V" H 1750 6040 50  0000 C CNN
 F 2 "" H 1750 5900 50  0001 C CNN
@@
 $EndComp
 $Comp
-L +5V #PWR041
+L +5V #PWR048
 U 1 1 5A04E6CC
 P 2500 4450
-F 0 "#PWR041" H 2500 4300 50  0001 C CNN
+F 0 "#PWR048" H 2500 4300 50  0001 C CNN
 F 1 "+5V" H 2500 4590 50  0000 C CNN
 F 2 "" H 2500 4450 50  0001 C CNN
@@
 5V Regulator\n
 $Comp
-L +5V #PWR042
+L +5V #PWR049
 U 1 1 5A05E9CE
 P 4200 6250
-F 0 "#PWR042" H 4200 6100 50  0001 C CNN
+F 0 "#PWR049" H 4200 6100 50  0001 C CNN
 F 1 "+5V" H 4200 6390 50  0000 C CNN
 F 2 "" H 4200 6250 50  0001 C CNN
@@
 $EndComp
 $Comp
-L GND #PWR043
+L GND #PWR050
 U 1 1 5A05F150
 P 4150 6750
-F 0 "#PWR043" H 4150 6500 50  0001 C CNN
+F 0 "#PWR050" H 4150 6500 50  0001 C CNN
 F 1 "GND" H 4150 6600 50  0000 C CNN
 F 2 "" H 4150 6750 50  0001 C CNN
@@
 $EndComp
 $Comp
-L +5V #PWR044
+L +5V #PWR051
 U 1 1 5A05FB12
 P 4150 7150
-F 0 "#PWR044" H 4150 7000 50  0001 C CNN
+F 0 "#PWR051" H 4150 7000 50  0001 C CNN
 F 1 "+5V" H 4150 7290 50  0000 C CNN
 F 2 "" H 4150 7150 50  0001 C CNN
@@
 	5800 6250 5950 6250
 $Comp
-L GND #PWR045
+L GND #PWR052
 U 1 1 5A0604B4
 P 5950 6550
-F 0 "#PWR045" H 5950 6300 50  0001 C CNN
+F 0 "#PWR052" H 5950 6300 50  0001 C CNN
 F 1 "GND" H 5950 6400 50  0000 C CNN
 F 2 "" H 5950 6550 50  0001 C CNN
@@
 $EndComp
 $Comp
-L GND #PWR046
+L GND #PWR053
 U 1 1 5A06054F
 P 5950 7450
-F 0 "#PWR046" H 5950 7200 50  0001 C CNN
+F 0 "#PWR053" H 5950 7200 50  0001 C CNN
 F 1 "GND" H 5950 7300 50  0000 C CNN
 F 2 "" H 5950 7450 50  0001 C CNN
@@
 $EndComp
 $Comp
-L +3.3V #PWR047
+L +3.3V #PWR054
 U 1 1 5A063648
 P 5950 6250
-F 0 "#PWR047" H 5950 6100 50  0001 C CNN
+F 0 "#PWR054" H 5950 6100 50  0001 C CNN
 F 1 "+3.3V" H 5950 6390 50  0000 C CNN
 F 2 "" H 5950 6250 50  0001 C CNN
@@
 $EndComp
 $Comp
-L GND #PWR048
+L GND #PWR055
 U 1 1 5A1CEE5F
 P 900 4650
-F 0 "#PWR048" H 900 4400 50  0001 C CNN
+F 0 "#PWR055" H 900 4400 50  0001 C CNN
 F 1 "GND" H 900 4500 50  0000 C CNN
 F 2 "" H 900 4650 50  0001 C CNN
@@
 Connection ~ 6200 2200
 $Comp
-L GND #PWR049
+L GND #PWR056
 U 1 1 5A1CF657
 P 6350 3250
-F 0 "#PWR049" H 6350 3000 50  0001 C CNN
+F 0 "#PWR056" H 6350 3000 50  0001 C CNN
 F 1 "GND" H 6350 3100 50  0000 C CNN
 F 2 "" H 6350 3250 50  0001 C CNN
@@
 $EndComp
 $Comp
-L GND #PWR050
+L GND #PWR057
 U 1 1 5A1CFAC3
 P 6350 4300
-F 0 "#PWR050" H 6350 4050 50  0001 C CNN
+F 0 "#PWR057" H 6350 4050 50  0001 C CNN
 F 1 "GND" H 6350 4150 50  0000 C CNN
 F 2 "" H 6350 4300 50  0001 C CNN
