File: Kicad Project/Radar.kicad_pcb (KiCad board)
At the start: 2 copper layers, 100 x 100 mm, 67 parts, among them J1 Conn_01x02, J2 Conn_01x02, J3 Conn_01x02, J4 Conn_01x02, J5 Conn_01x02, J6 Conn_01x02, J7 Conn_01x02, U1 GALI-1+, U10 GALI-2+, U11 BandpassFilter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

Commit message: Changed Routing of 9V line, added more documentation
Routing:
- net +9V: track 148.7 -> 298.1 mm, vias 2 -> 0
Changed lines of the file:
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@@
   (general
     (links 186)
-    (no_connects 14)
+    (no_connects 13)
     (area 79.0194 73.0758 201.345801 179.146201)
     (thickness 1.6)
     (drawings 4)
-    (tracks 387)
+    (tracks 390)
     (zones 0)
     (modules 67)
@@
   )
   (setup
-    (last_trace_width 0.381)
+    (last_trace_width 0.508)
     (user_trace_width 0.254)
     (user_trace_width 0.381)
@@
   (segment (start 122.2013 124.1806) (end 122.2013 130.0734) (width 2.54) (layer F.Cu) (net 11))
   (segment (start 186.58776 123.4313) (end 186.58776 126.91364) (width 2.54) (layer F.Cu) (net 12))
+  (segment (start 172.4552 134.0866) (end 154.305 134.0866) (width 0.508) (layer F.Cu) (net 13))
+  (segment (start 102.1969 127.127) (end 107.69282 127.127) (width 0.508) (layer F.Cu) (net 13))
+  (segment (start 96.901 132.4229) (end 102.1969 127.127) (width 0.508) (layer F.Cu) (net 13))
+  (segment (start 96.901 170.1673) (end 96.901 132.4229) (width 0.508) (layer F.Cu) (net 13))
+  (segment (start 100.6856 173.9519) (end 96.901 170.1673) (width 0.508) (layer F.Cu) (net 13))
+  (segment (start 138.303 173.9519) (end 100.6856 173.9519) (width 0.508) (layer F.Cu) (net 13))
+  (segment (start 148.3106 163.9443) (end 138.303 173.9519) (width 0.508) (layer F.Cu) (net 13))
+  (segment (start 148.3106 140.081) (end 148.3106 163.9443) (width 0.508) (layer F.Cu) (net 13))
+  (segment (start 154.305 134.0866) (end 148.3106 140.081) (width 0.508) (layer F.Cu) (net 13))
+  (segment (start 131.288543 112.5594) (end 119.2777 112.5594) (width 0.25) (layer F.Cu) (net 13))
+  (segment (start 118.43956 111.72126) (end 118.43956 106.807) (width 0.25) (layer F.Cu) (net 13))
+  (segment (start 119.2777 112.5594) (end 118.43956 111.72126) (width 0.25) (layer F.Cu) (net 13))
   (segment (start 99.2016 113.8682) (end 99.2016 118.0738) (width 0.762) (layer F.Cu) (net 13))
   (segment (start 103.2026 122.0748) (end 107.3936 122.0748) (width 0.762) (layer F.Cu) (net 13))
   (segment (start 99.2016 118.0738) (end 103.2026 122.0748) (width 0.762) (layer F.Cu) (net 13))
-  (segment (start 170.05236 112.93856) (end 172.17136 112.93856) (width 0.508) (layer F.Cu) (net 13))
-  (segment (start 172.4552 128.9666) (end 172.4552 134.0866) (width 0.508) (layer F.Cu) (net 13))
-  (segment (start 176.784 124.6378) (end 172.4552 128.9666) (width 0.508) (layer F.Cu) (net 13))
-  (via (at 176.784 124.6378) (size 0.6) (drill 0.4) (layers F.Cu B.Cu) (net 13))
-  (segment (start 176.784 120.2436) (end 176.784 124.6378) (width 0.508) (layer B.Cu) (net 13))
-  (segment (start 176.8094 120.2182) (end 176.784 120.2436) (width 0.508) (layer B.Cu) (net 13))
-  (via (at 176.8094 120.2182) (size 0.6) (drill 0.4) (layers F.Cu B.Cu) (net 13))
-  (segment (start 176.8094 117.5766) (end 176.8094 120.2182) (width 0.508) (layer F.Cu) (net 13))
-  (segment (start 172.17136 112.93856) (end 176.8094 117.5766) (width 0.508) (layer F.Cu) (net 13))
   (segment (start 107.3936 111.5822) (end 107.3936 109.9288) (width 1.27) (layer F.Cu) (net 13))
   (segment (start 130.4544 104.267) (end 137.62164 104.267) (width 1.27) (layer F.Cu) (net 13))

Commit message: PCB Edits post PDR
Parts:
- added ?: , RadarComponents:Via, F.Cu at (144.2, 98.3)
- added ?: , RadarComponents:Via, F.Cu at (154.0, 120.1)
- added ?: , RadarComponents:Via, F.Cu at (152.7, 120.1)
- added ?: , RadarComponents:Via, F.Cu at (151.5, 120.1)
- added ?: , RadarComponents:Via, F.Cu at (155.3, 118.8)
- added ?: , RadarComponents:Via, F.Cu at (154.0, 118.8)
- added ?: , RadarComponents:Via, F.Cu at (152.7, 118.8)
- added ?: , RadarComponents:Via, F.Cu at (151.5, 118.8)
- added ?: , RadarComponents:LOGO, F.Cu at (146.8, 158.5)
- added ?: , RadarComponents:Via, F.Cu at (143.0, 98.3)
- added ?: , RadarComponents:Via, F.Cu at (141.7, 98.3)
- added ?: , RadarComponents:Via, F.Cu at (140.4, 98.3)
- added ?: , RadarComponents:Via, F.Cu at (144.2, 97.0)
- added ?: , RadarComponents:Via, F.Cu at (143.0, 97.0)
- added ?: , RadarComponents:Via, F.Cu at (141.7, 97.0)
- added ?: , RadarComponents:Via, F.Cu at (140.4, 97.0)
- added ?: , RadarComponents:Via, F.Cu at (155.3, 120.1)
- added C22: 1uF, Capacitors_SMD:C_0805, F.Cu at (103.5, 100.0)
- added C23: 470pF, Capacitors_SMD:C_0805, F.Cu at (112.1, 101.0)
- added R21: 51, Resistors_SMD:R_0603, F.Cu at (154.9, 113.4)
- added R22: 2K, Resistors_SMD:R_0603, F.Cu at (101.3, 83.3)
- added R23: 2K, Resistors_SMD:R_0603, F.Cu at (104.2, 84.0)
- added U16: TC1185, RadarComponents:SOT23-5, F.Cu at (106.7, 101.2)
- C15, C4: value 270pF -> ?F
- C18, C20, C21: value C -> 10nF
- moved J4 1.77 mm to (131.0, 85.1), turned to 90 degrees
Connections:
- C16 pad 1: +9V -> +3V3
- J4 pad 1: GND -> Net-(J4-Pad1)
- J4 pad 2: Net-(J4-Pad2) -> GND
- R10 pad 2: Net-(J4-Pad2) -> Net-(J4-Pad1)
- R11 pad 1: Net-(J4-Pad2) -> Net-(J4-Pad1)
- U2 pad 2: GND -> (no net)
- U2 pad 4: GND -> (no net)
- U2 pad 6: GND -> (no net)
- U2 pad 7: GND -> (no net)
- U2 pad 8: GND -> (no net)
- U2 pad 9: GND -> (no net)
- U4 pad 5: +9V -> +3V3
- VCO1 pad 2: Net-(J1-Pad2) -> Net-(R22-Pad1)
Routing:
- net +3V3: track 4.55 -> 79.8 mm, vias 0 -> 4
- net Net-(J1-Pad2): track 0.00 -> 28.1 mm
- net Net-(J7-Pad2): track 0.00 -> 18.5 mm
- net Net-(J4-Pad2): track 12.9 -> 0.00 mm
- net Net-(J4-Pad1): track 0.00 -> 12.9 mm
- net +5V: track 32.9 -> 44.6 mm
- net +9V: track 298.1 -> 306.8 mm
- net Net-(R22-Pad1): track 0.00 -> 6.89 mm
- net GND: track 139.4 -> 143.3 mm, vias 52 -> 44
- net Net-(C23-Pad1): track 0.00 -> 2.88 mm
- net Net-(C15-Pad2): track 10.3 -> 11.7 mm
Other:
- board text added: "Generic Radar Organization Katie Dhuyvetter Thomas Gorham Nathan Jones Damian Loya"

Commit message: updated gerbers
Parts:
- moved .1uF4 24.6 mm to (161.9, 78.3)
- moved ? 24.6 mm to (141.0, 99.2)
- moved ? 24.6 mm to (128.7, 77.4)
- moved ? 24.6 mm to (128.7, 76.1)
- moved C21 24.6 mm to (145.4, 78.3)
- moved R14 24.6 mm to (155.8, 90.1)
- moved ? 24.6 mm to (141.0, 97.9)
- moved ? 24.6 mm to (127.4, 77.4)
- moved ? 24.6 mm to (127.4, 76.1)
- moved C1 24.6 mm to (163.5, 102.8)
- moved C10 24.6 mm to (110.5, 102.0)
- moved C11 24.6 mm to (174.9, 101.2)
- moved C16 24.6 mm to (123.9, 87.6)
- moved C5 24.6 mm to (91.3, 67.7)
- moved C8 24.6 mm to (106.7, 80.9)
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
Commit message: Rev 1!
Gerbers Generated
Sent to Smart
Parts:
- removed R15: R, Resistors_SMD:R_0603
- added 0ohms1, 0ohms2: R, RadarComponents:100PAD, F.Cu at (131.4, 165.5)
- C10, C11, C12, C13, C14: value 150p -> 100n
Connections:
- U5 pad 1: Net-(R15-Pad1) -> GND
- U7 pad 3: GND -> (no net)
- U7 pad 5: GND -> (no net)
- U7 pad 6: GND -> (no net)
Routing:
- net Net-(R15-Pad1): track 5.45 -> 0.01 mm
- net GND: track 143.3 -> 143.9 mm
Changed lines of the file:
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@@
 (kicad_pcb (version 4) (host pcbnew 4.0.7)
   (general
-    (links 209)
+    (links 204)
     (no_connects 10)
-    (area 79.0194 73.0758 201.345801 179.146201)
+    (area 81.310199 55.355399 181.460201 155.505401)
     (thickness 1.6)
     (drawings 5)
-    (tracks 439)
+    (tracks 435)
     (zones 0)
-    (modules 90)
-    (nets 43)
+    (modules 91)
+    (nets 47)
   )
   (page A4)
@@
     (pad_to_mask_clearance 0.2)
     (aux_axis_origin 0 0)
-    (grid_origin 154.0002 120.1166)
+    (grid_origin 89.9668 115.0366)
     (visible_elements 7FFFFFFF)
     (pcbplotparams
-      (layerselection 0x00030_80000001)
+      (layerselection 0x000f0_80000001)
       (usegerberextensions false)
       (excludeedgelayer true)
@@
   (net 41 "Net-(J4-Pad1)")
   (net 42 "Net-(R22-Pad1)")
+  (net 43 "Net-(0ohms1-Pad2)")
+  (net 44 "Net-(0ohms1-Pad1)")
+  (net 45 "Net-(0ohms2-Pad2)")
+  (net 46 "Net-(0ohms2-Pad1)")
   (net_class Default "This is the default net class."
     (clearance 0.2)
@@
     (add_net "Net-(.1uF4-Pad1)")
     (add_net "Net-(.1uF4-Pad2)")
+    (add_net "Net-(0ohms1-Pad1)")
+    (add_net "Net-(0ohms1-Pad2)")
+    (add_net "Net-(0ohms2-Pad1)")
+    (add_net "Net-(0ohms2-Pad2)")
     (add_net "Net-(C1-Pad1)")
     (add_net "Net-(C10-Pad1)")
@@
     (pad 2 smd rect (at 3.3274 -0.8382) (size 1.524 1.651) (layers F.Cu F.Paste F.Mask)
       (net 4 GND))
-    (pad 3 smd rect (at 5.8674 -0.8382) (size 1.524 1.651) (layers F.Cu F.Paste F.Mask)
-      (net 4 GND))
-    (pad 6 smd rect (at 0.7874 5.1308) (size 1.524 1.651) (layers F.Cu F.Paste F.Mask)
-      (net 4 GND))
-    (pad 5 smd rect (at 3.3274 5.1308) (size 1.524 1.651) (layers F.Cu F.Paste F.Mask)
-      (net 4 GND))
+    (pad 3 smd rect (at 5.8674 -0.8382) (size 1.524 1.651) (layers F.Cu F.Paste F.Mask))
+    (pad 6 smd rect (at 0.7874 5.1308) (size 1.524 1.651) (layers F.Cu F.Paste F.Mask))
+    (pad 5 smd rect (at 3.3274 5.1308) (size 1.524 1.651) (layers F.Cu F.Paste F.Mask))
     (pad 1 smd rect (at 0.3048 -0.8636) (size 2.54 2.54) (layers F.Cu F.Paste F.Mask)
       (net 16 "Net-(R12-Pad1)"))
@@
       (effects (font (size 1 1) (thickness 0.15)))
     )
-    (fp_text value 150p (at 5.842 -3.683 90) (layer F.Fab)
+    (fp_text value 100n (at 5.842 -3.683 90) (layer F.Fab)
       (effects (font (size 1 1) (thickness 0.15)))
     )
@@
       (effects (font (size 1 1) (thickness 0.15)))
     )
-    (fp_text value 150p (at 5.842 -3.683 90) (layer F.Fab)
+    (fp_text value 100n (at 5.842 -3.683 90) (layer F.Fab)
       (effects (font (size 1 1) (thickness 0.15)))
     )
@@
       (effects (font (size 1 1) (thickness 0.15)))
     )
-    (fp_text value 150p (at 5.842 -3.683 90) (layer F.Fab)
+    (fp_text value 100n (at 5.842 -3.683 90) (layer F.Fab)
       (effects (font (size 1 1) (thickness 0.15)))
     )
@@
   )
   (module Resistors_SMD:R_0603 (layer F.Cu)
-    (at 88.2669 95.70212 270)
-    (descr "Resistor SMD 0603, reflow soldering, Vishay (see dcrcw.pdf)")
-    (tags "resistor 0603")
-    (attr smd)
-    (fp_text reference R15 (at 0 -1.45 270) (layer F.SilkS)
-      (effects (font (size 1 1) (thickness 0.15)))
-    )
-    (fp_text value R (at 0 1.5 270) (layer F.Fab)
-      (effects (font (size 1 1) (thickness 0.15)))
-    )
-    (fp_text user %R (at 0 0 270) (layer F.Fab)
-      (effects (font (size 0.4 0.4) (thickness 0.075)))
-    )
-    (fp_line (start -0.8 0.4) (end -0.8 -0.4) (layer F.Fab) (width 0.1))
-    (fp_line (start 0.8 0.4) (end -0.8 0.4) (layer F.Fab) (width 0.1))
-    (fp_line (start 0.8 -0.4) (end 0.8 0.4) (layer F.Fab) (width 0.1))
-    (fp_line (start -0.8 -0.4) (end 0.8 -0.4) (layer F.Fab) (width 0.1))
-    (fp_line (start 0.5 0.68) (end -0.5 0.68) (layer F.SilkS) (width 0.12))
-    (fp_line (start -0.5 -0.68) (end 0.5 -0.68) (layer F.SilkS) (width 0.12))
-    (fp_line (start -1.25 -0.7) (end 1.25 -0.7) (layer F.CrtYd) (width 0.05))
-    (fp_line (start -1.25 -0.7) (end -1.25 0.7) (layer F.CrtYd) (width 0.05))
-    (fp_line (start 1.25 0.7) (end 1.25 -0.7) (layer F.CrtYd) (width 0.05))
-    (fp_line (start 1.25 0.7) (end -1.25 0.7) (layer F.CrtYd) (width 0.05))
-    (pad 1 smd rect (at -0.75 0 270) (size 0.5 0.9) (layers F.Cu F.Paste F.Mask)
-      (net 20 "Net-(R15-Pad1)"))
-    (pad 2 smd rect (at 0.75 0 270) (size 0.5 0.9) (layers F.Cu F.Paste F.Mask)
-      (net 4 GND))
-    (model ${KISYS3DMOD}/Resistors_SMD.3dshapes/R_0603.wrl
-      (at (xyz 0 0 0))
-      (scale (xyz 1 1 1))
-      (rotate (xyz 0 0 0))
-    )
-  )
-  (module Resistors_SMD:R_0603 (layer F.Cu)
     (at 89.79852 93.38056 90)
     (descr "Resistor SMD 0603, reflow soldering, Vishay (see dcrcw.pdf)")
@@
       (net 30 +5V))
     (pad 1 smd rect (at -2.25 0) (size 1.2 1.6) (layers F.Cu F.Paste F.Mask)
-      (net 20 "Net-(R15-Pad1)"))
+      (net 4 GND))
     (pad 2 smd rect (at 0 0) (size 1.2 1.6) (layers F.Cu F.Paste F.Mask)
       (net 30 +5V))
@@
       (effects (font (size 1 1) (thickness 0.15)))
     )
-    (fp_text value 150p (at 5.842 -3.683 270) (layer F.Fab)
+    (fp_text value 100n (at 5.842 -3.683 270) (layer F.Fab)
       (effects (font (size 1 1) (thickness 0.15)))
     )
@@
       (effects (font (size 1 1) (thickness 0.15)))
     )
-    (fp_text value 150p (at 5.842 -3.683 270) (layer F.Fab)
+    (fp_text value 100n (at 5.842 -3.683 270) (layer F.Fab)
       (effects (font (size 1 1) (thickness 0.15)))
     )
@@
       (xy 8.592538 -10.079684) (xy 8.655653 -10.039906)) (layer F.SilkS) (width 0.01))
   )
+  (module RadarComponents:100PAD (layer F.Cu)
+    (at 131.3852 165.505401)
+    (fp_text reference 0ohms1 (at 1.143 -3.3274) (layer F.SilkS)
+      (effects (font (size 1 1) (thickness 0.15)))
+    )
+    (fp_text value R (at 0.3048 0.7112) (layer F.Fab)
+      (effects (font (size 1 1) (thickness 0.15)))
+    )
+    (pad 2 smd rect (at 1.9304 -1.27) (size 2.54 2.54) (layers F.Cu F.Paste F.Mask)
+      (net 43 "Net-(0ohms1-Pad2)"))
+    (pad 1 smd rect (at -1.27 -1.27) (size 2.54 2.54) (layers F.Cu F.Paste F.Mask)
+      (net 44 "Net-(0ohms1-Pad1)"))
+  )
+  (module RadarComponents:100PAD (layer F.Cu)
+    (at 131.3852 165.505401)
+    (fp_text reference 0ohms2 (at 1.143 -3.3274) (layer F.SilkS)
+      (effects (font (size 1 1) (thickness 0.15)))
+    )
+    (fp_text value R (at 0.3048 0.7112) (layer F.Fab)
+      (effects (font (size 1 1) (thickness 0.15)))
+    )
+    (pad 2 smd rect (at 1.9304 -1.27) (size 2.54 2.54) (layers F.Cu F.Paste F.Mask)
+      (net 45 "Net-(0ohms2-Pad2)"))
+    (pad 1 smd rect (at -1.27 -1.27) (size 2.54 2.54) (layers F.Cu F.Paste F.Mask)
+      (net 46 "Net-(0ohms2-Pad1)"))
+  )
   (gr_text "Generic Radar Organization\n\nKatie Dhuyvetter\nThomas Gorham\nNathan Jones\nDamian Loya" (at 134.1247 118.2624) (layer F.SilkS)
     (effects (font (size 1.5 1.5) (thickness 0.3)))
@@
   (segment (start 150.1032 94.69628) (end 150.1032 98.30816) (width 2.54) (layer F.Cu) (net 3))
   (segment (start 150.1032 98.30816) (end 150.10828 98.31324) (width 2.54) (layer F.Cu) (net 3))
+  (segment (start 89.7888 90.6526) (end 88.83396 90.6526) (width 0.25) (layer F.Cu) (net 4) (status 400000))
+  (via (at 88.21928 91.26728) (size 0.6) (drill 0.4) (layers F.Cu B.Cu) (net 4))
+  (segment (start 88.83396 90.6526) (end 88.21928 91.26728) (width 0.25) (layer F.Cu) (net 4))
   (segment (start 141.9225 98.7806) (end 141.9225 98.806) (width 0.508) (layer B.Cu) (net 4))
   (segment (start 141.9098 98.7679) (end 141.9225 98.7806) (width 0.508) (layer B.Cu) (net 4))
@@
   (via (at 91.9734 96.5073) (size 0.6) (drill 0.4) (layers F.Cu B.Cu) (net 4))
   (segment (start 92.0388 96.4419) (end 91.9734 96.5073) (width 0.381) (layer F.Cu) (net 4))
-  (segment (start 88.2669 96.45212) (end 89.41632 96.45212) (width 0.381) (layer F.Cu) (net 4))
-  (via (at 89.4715 96.5073) (size 0.6) (drill 0.4) (layers F.Cu B.Cu) (net 4))
-  (segment (start 89.41632 96.45212) (end 89.4715 96.5073) (width 0.381) (layer F.Cu) (net 4))
   (via (at 123.992 60.1218) (size 0.6) (drill 0.4) (layers F.Cu B.Cu) (net 4))
   (segment (start 90.9339 132.1921) (end 89.334 132.1921) (width 0.508) (layer F.Cu) (net 4))
@@
   (segment (start 173.5728 119.33936) (end 173.5728 123.06046) (width 2.54) (layer F.Cu) (net 19))
   (segment (start 173.5728 123.06046) (end 173.57534 123.063) (width 2.54) (layer F.Cu) (net 19))
-  (segment (start 88.2669 94.95212) (end 88.2669 93.29166) (width 0.508) (layer F.Cu) (net 20))
-  (segment (start 88.928 92.63056) (end 89.79852 92.63056) (width 0.508) (layer F.Cu) (net 20))
-  (segment (start 88.2669 93.29166) (end 88.928 92.63056) (width 0.508) (layer F.Cu) (net 20))
-  (segment (start 89.7888 90.6526) (end 89.7888 92.62084) (width 0.508) (layer F.Cu) (net 20))
   (segment (start 89.7888 92.62084) (end 89.79852 92.63056) (width 0.508) (layer F.Cu) (net 20))
   (segment (start 173.5855 97.0026) (end 173.5855 99.29876) (width 2.54) (layer F.Cu) (net 21))
